Commit message: Update URDF with accurate GoGoPi dimensions: 133x95x31mm body, 67mm drive wheels, ball castor, 89mm sensor tower

File: ros2/src/gogopi_bringup/urdf/gogopi.urdf (robot description, URDF)
Before this commit: robot gogopi, 10 links, 9 joints
Links:
- removed link wheel_rear_left
- removed link wheel_rear_right
- added link castor_link, mass 0.05; collision sphere radius=0.01; visual sphere radius=0.01
- link base_link: geometry collision box size=0.133 0.095 0.031; visual box size=0.133 0.095 0.031
- link sensor_tower: geometry collision box size=0.002 0.055 0.089; visual box size=0.002 0.055 0.089
- link wheel_front_left: geometry collision cylinder length=0.021 radius=0.0335; visual cylinder length=0.021 radius=0.0335
- link wheel_front_right: geometry collision cylinder length=0.021 radius=0.0335; visual cylinder length=0.021 radius=0.0335
Joints:
- removed joint wheel_rear_left_joint
- removed joint wheel_rear_right_joint
- added joint castor_joint: type fixed, parent base_link, child castor_link, origin xyz=-0.0545 0 0.01 rpy=0 0 0
- joint pan_joint: origin xyz=0 0 0.2 rpy=0 0 0 -> xyz=0 0 0.089 rpy=0 0 0
- joint sensor_tower_joint: origin xyz=0 0 0.15 rpy=0 0 0 -> xyz=-0.0475 0 0.06 rpy=0 0 0
- joint wheel_front_left_joint: origin xyz=0.075 0.075 0 rpy=0 0 0 -> xyz=0.0295 0.083 0 rpy=0 0 0
- joint wheel_front_right_joint: origin xyz=0.075 -0.075 0 rpy=0 0 0 -> xyz=0.0295 -0.083 0 rpy=0 0 0

Commit message: Add athe cameras to the tilt arm

File: ros2/src/gogopi_bringup/urdf/gogopi.urdf (robot description, URDF)
Before this commit: robot gogopi, 9 links, 8 joints
Links:
- link camera_link: geometry collision box size=0.017 0.025 0.030; visual box size=0.002 0.025 0.030
- link pan_link: geometry collision cylinder length=0.005 radius=0.021; visual cylinder length=0.005 radius=0.021
- link sensor_tower: geometry collision box size=0.002 0.055 0.089; visual box size=0.002 0.055 0.089
- link thermal_camera_link: geometry collision box size=0.012 0.015 0.026; visual box size=0.002 0.015 0.026
- link tilt_link: geometry collision box size=0.036 0.040 0.013; visual box size=0.036 0.040 0.013
Joints:
- joint camera_joint: origin xyz=0.025 0 0 rpy=0 0 0 -> xyz=0.019 0.0075 0 rpy=0 0 0
- joint pan_joint: origin xyz=0 0 0.089 rpy=0 0 0 -> xyz=0.026 0 0.092 rpy=0 0 0
- joint sensor_tower_joint: origin xyz=-0.0475 0 0.06 rpy=0 0 0 -> xyz=-0.0475 0 0.031 rpy=0 0 0
- joint thermal_camera_joint: origin xyz=0.025 0.03 0 rpy=0 0 0 -> xyz=0.020 -0.0125 0.013 rpy=0 0 0
- joint tilt_joint: origin xyz=0.025 0 0 rpy=0 0 0 -> xyz=-0.012 0 0.0235 rpy=0 0 0

Commit message: Rotate the lidar in the URDF to point consistently

File: ros2/src/gogopi_bringup/urdf/gogopi.urdf (robot description, URDF)
Before this commit: robot gogopi, 11 links, 10 joints
Joints:
- joint lidar_joint: origin xyz=0.0295 0 0.0965 rpy=0 0 0 -> xyz=0.0295 0 0.0965 rpy=0 0 3.14159
