Commit message: Fix URDF wheel orientation, castor geometry, and wheel separation
- Rotate drive wheels 90° (rpy 1.5708 0 0) so cylinders face Y axis
- Move wheels to ±60mm (2mm gap from 95mm-wide body)
- Update wheel_separation_m default to 0.12 in board_node
- Fix castor: 14mm silver sphere, black 22mm cylindrical mount
- Add test_urdf.launch.py for publishing robot_description over network

Co-Authored-By: Claude Sonnet 4.6 <noreply@anthropic.com>

File: ros2/src/gogopi_bringup/urdf/gogopi.urdf (robot description, URDF)
Before this commit: robot gogopi, 9 links, 8 joints
Links:
- link castor_link: geometry collision sphere radius=0.007; visual cylinder length=0.0195 radius=0.011
Joints:
- joint castor_joint: origin xyz=-0.0545 0 0.01 rpy=0 0 0 -> xyz=-0.0545 0 -0.0265 rpy=0 0 0
- joint wheel_front_left_joint: origin xyz=0.0295 0.083 0 rpy=0 0 0 -> xyz=0.0295 0.060 0 rpy=0 0 0
- joint wheel_front_right_joint: origin xyz=0.0295 -0.083 0 rpy=0 0 0 -> xyz=0.0295 -0.060 0 rpy=0 0 0

Commit message: Add YDLidar TX lidar node and URDF placement
lidar_node.py: lifecycle node wrapping the YDLidar Python SDK.
Background thread runs the blocking scan loop; a timer on the
executor thread drains the queue and publishes sensor_msgs/LaserScan
on /gogopi/lidar/scan at 7 Hz with 1° angular resolution.

URDF: lidar_link (80mm dia × 15mm cylinder) fixed at wheel-axis x,
robot centreline y, 130mm above floor (z=0.0965 in base_link).

gprctl: window 6 for lidar_node (/dev/ttyUSB0 check), window 7 for
shell; lidar_node added to auto-lifecycle sequence.

Co-Authored-By: Claude Sonnet 4.6 <noreply@anthropic.com>

File: ros2/src/gogopi_bringup/urdf/gogopi.urdf (robot description, URDF)
Before this commit: robot gogopi, 9 links, 8 joints
Links:
- added link lidar_link, mass 0.08; collision cylinder length=0.015 radius=0.040; visual cylinder length=0.015 radius=0.040
Joints:
- added joint lidar_joint: type fixed, parent base_link, child lidar_link, origin xyz=0.0295 0 0.0965 rpy=0 0 0

Commit message: RViz on quattro: LAN/Tailscale discovery, real-servo TF, sensor displays
- run.sh: use the Tailscale unicast-peer profile only when Tailscale is up;
  otherwise plain LAN multicast (with the peer profile and Tailscale down,
  nothing was discovered)
- container no longer runs its own robot_state_publisher (duplicate TF);
  joint_state_publisher_gui reads /robot_description from the robot
- test_urdf.launch.py (gprctl urdf window): remap /joint_states →
  /gogopi/servo_state like robot.launch.py, so TF follows the real servos
- URDF: sonar_link (placeholder pose; module not mounted yet)
- default.rviz: add Camera, Lidar (LaserScan), Sonar (Range) displays;
  RobotModel description topic Transient Local so it gets the latched URDF

Co-Authored-By: Claude Opus 5.5 <noreply@anthropic.com>

File: ros2/src/gogopi_bringup/urdf/gogopi.urdf (robot description, URDF)
Before this commit: robot gogopi, 11 links, 10 joints
Links:
- added link sonar_link
Joints:
- added joint sonar_joint: type fixed, parent base_link, child sonar_link, origin xyz=0.0665 0 0.0155 rpy=0 0 0

Commit message: URDF: sonar_link on rear face of sensor tower, facing backward, 100 mm up
Co-Authored-By: Claude Opus 5.5 <noreply@anthropic.com>

File: ros2/src/gogopi_bringup/urdf/gogopi.urdf (robot description, URDF)
Before this commit: robot gogopi, 12 links, 11 joints
Joints:
- joint sonar_joint: origin xyz=0.0665 0 0.0155 rpy=0 0 0 -> xyz=-0.016 0 0.0355 rpy=0 0 3.14159; parent base_link -> sensor_tower

Commit message: URDF: tilt zero pose is 45° up (measured with sliders centred)
Co-Authored-By: Claude Opus 5.5 <noreply@anthropic.com>

File: ros2/src/gogopi_bringup/urdf/gogopi.urdf (robot description, URDF)
Before this commit: robot gogopi, 12 links, 11 joints
Joints:
- joint tilt_joint: origin xyz=-0.012 0 0.0235 rpy=0 0 0 -> xyz=-0.012 0 0.0235 rpy=0 -0.7854 0

Commit message: board_node: clamp servo commands to mechanical travel; URDF limits
Tilt hits its low stop at servo ~13.8° (slider 1.33 rad) and stalled there,
jittering on USB power. New params servo_min_deg/servo_max_deg ([17,0] /
[180,180]) clamp every command path (angle, pulse, /joint_states).
URDF: tilt upper limit 1.2741 rad (= servo 17°), pan ±90° to match the
servo's 0–180° (slider allowed ±180°).

Co-Authored-By: Claude Opus 5.5 <noreply@anthropic.com>

File: ros2/src/gogopi_bringup/urdf/gogopi.urdf (robot description, URDF)
Before this commit: robot gogopi, 12 links, 11 joints
Joints:
- joint pan_joint: limit lower=-3.14159 upper=3.14159 effort=1.0 velocity=1.0 -> lower=-1.5708 upper=1.5708 effort=1.0 velocity=1.0
- joint tilt_joint: limit lower=-1.5708 upper=1.5708 effort=1.0 velocity=1.0 -> lower=-1.5708 upper=1.2741 effort=1.0 velocity=1.0

Commit message: Tilt practical max = servo 90° (camera 45° up): panning binds cables above it
Camera sweep: tilt moves freely 90→180° (no stop), but with significant
pan, tilt beyond the centre position binds the cables. servo_max_deg
[90, 180]; URDF tilt_joint lower 0.0.

Co-Authored-By: Claude Opus 5.5 <noreply@anthropic.com>

File: ros2/src/gogopi_bringup/urdf/gogopi.urdf (robot description, URDF)
Before this commit: robot gogopi, 12 links, 11 joints
Joints:
- joint tilt_joint: limit lower=-1.5708 upper=1.2741 effort=1.0 velocity=1.0 -> lower=0.0 upper=1.2741 effort=1.0 velocity=1.0

Commit message: Tilt calibrated: level = servo 28°, 0.66° per commanded degree
pan-check (image twist while panning) crosses zero between servo 26° and
29°; pitch changes ~0.66° per commanded degree (cheap SG9), so servo 90°
points ~41° up — matching the earlier visual '≈45° up'.

board_node: new params joint_zero_servo_deg [28, 90] and
joint_deg_per_servo_deg [0.66, 1.0] drive both servo_state and the
/joint_states inverse. URDF: tilt_joint 0 = level (origin pitch 0), limits
−0.7142 … 0.1267 rad for the 90°/17° clamps. pt_range_check levels the
camera at 28° for pan. Cheat sheet: level = 28°.

Co-Authored-By: Claude Opus 5.5 <noreply@anthropic.com>

File: ros2/src/gogopi_bringup/urdf/gogopi.urdf (robot description, URDF)
Before this commit: robot gogopi, 12 links, 11 joints
Joints:
- joint tilt_joint: limit lower=0.0 upper=1.2741 effort=1.0 velocity=1.0 -> lower=-0.7142 upper=0.1267 effort=1.0 velocity=1.0; origin xyz=-0.012 0 0.0235 rpy=0 -0.7854 0 -> xyz=-0.012 0 0.0235 rpy=0 0 0

Commit message: Tilt scale 1.08°/commanded° (inclinometer: servo 90° ≈ 67° up); pan 1.0
Focal length from the shelf (85 cm outside-outside at 3 m → 172–176 px →
f ≈ 612 px) plus image shift per degree gave tilt 1.13 / pan 1.0; an
inclinometer at servo 90° read ~67° (62 commanded ° above level) → 1.08.
The earlier 0.66 came from assuming pan-check's slope = s_tilt·s_pan, which
doesn't hold here. URDF tilt limits −1.1687 … 0.2073 rad.

Co-Authored-By: Claude Opus 5.5 <noreply@anthropic.com>

File: ros2/src/gogopi_bringup/urdf/gogopi.urdf (robot description, URDF)
Before this commit: robot gogopi, 12 links, 11 joints
Joints:
- joint tilt_joint: limit lower=-0.7142 upper=0.1267 effort=1.0 velocity=1.0 -> lower=-1.1687 upper=0.2073 effort=1.0 velocity=1.0

Commit message: Pan temporarily limited to 40–140° until the tower wiring is rerouted
Hard pan swings during tools/pt_lidar_stress.py snapped one of the camera's USB
data wires at its connector (after several −71 / full-speed dropouts). servo
limits [17, 40] … [90, 140]; URDF pan_joint ±0.8727 rad.

Co-Authored-By: Claude Opus 5.5 <noreply@anthropic.com>

File: ros2/src/gogopi_bringup/urdf/gogopi.urdf (robot description, URDF)
Before this commit: robot gogopi, 12 links, 11 joints
Joints:
- joint pan_joint: limit lower=-1.5708 upper=1.5708 effort=1.0 velocity=1.0 -> lower=-0.8727 upper=0.8727 effort=1.0 velocity=1.0

Commit message: URDF: wheels 1 mm outside the frame (y ±0.059)
Co-Authored-By: Claude Opus 5.5 <noreply@anthropic.com>

File: ros2/src/gogopi_bringup/urdf/gogopi.urdf (robot description, URDF)
Before this commit: robot gogopi, 12 links, 11 joints
Joints:
- joint wheel_front_left_joint: origin xyz=0.0295 0.060 0 rpy=0 0 0 -> xyz=0.0295 0.059 0 rpy=0 0 0
- joint wheel_front_right_joint: origin xyz=0.0295 -0.060 0 rpy=0 0 0 -> xyz=0.0295 -0.059 0 rpy=0 0 0

Commit message: URDF: fixed wheel joints so they get a TF
No wheel encoders, and robot_state_publisher only gets /gogopi/servo_state
(pan/tilt), so the continuous wheel joints never had a transform and RViz
drew both wheels at the base_link origin.

Co-Authored-By: Claude Opus 5.5 <noreply@anthropic.com>

File: ros2/src/gogopi_bringup/urdf/gogopi.urdf (robot description, URDF)
Before this commit: robot gogopi, 12 links, 11 joints
Joints:
- joint wheel_front_left_joint: axis 0 1 0 -> (none); type continuous -> fixed
- joint wheel_front_right_joint: axis 0 1 0 -> (none); type continuous -> fixed

Commit message: URDF: base_footprint on the floor; RViz fixed frame base_footprint
Raise base_link 33.5 mm above base_footprint so the wheel bottoms and the
castor ball touch z = 0, and use base_footprint as the RViz fixed frame so
the grid is the floor.

Co-Authored-By: Claude Opus 5.5 <noreply@anthropic.com>

File: ros2/src/gogopi_bringup/urdf/gogopi.urdf (robot description, URDF)
Before this commit: robot gogopi, 12 links, 11 joints
Joints:
- joint base_footprint_joint: origin xyz=0 0 0 rpy=0 0 0 -> xyz=0 0 0.0335 rpy=0 0 0
